Commit message: Reference the same button dae

File: assets/elevator2.urdf (robot description, URDF)
Before this commit: robot elevator, 10 links, 9 joints
Links:
- link button_0_0_link: geometry collision box size=0.19 0.02 0.09; visual mesh filename=button.dae scale=1 1 1
- link button_0_1_link: geometry collision box size=0.19 0.02 0.09; visual mesh filename=button.dae scale=1 1 1
- link button_1_0_link: geometry collision box size=0.19 0.02 0.09; visual mesh filename=button.dae scale=1 1 1
- link button_1_1_link: geometry collision box size=0.19 0.02 0.09; visual mesh filename=button.dae scale=1 1 1
- link button_2_0_link: geometry collision box size=0.19 0.02 0.09; visual mesh filename=button.dae scale=1 1 1
- link button_2_1_link: geometry collision box size=0.19 0.02 0.09; visual mesh filename=button.dae scale=1 1 1
- link button_3_0_link: geometry collision box size=0.19 0.02 0.09; visual mesh filename=button.dae scale=1 1 1
- link button_3_1_link: geometry collision box size=0.19 0.02 0.09; visual mesh filename=button.dae scale=1 1 1

Commit message: Fix URDF

File: assets/elevator2.urdf (robot description, URDF)
Before this commit: robot elevator, 10 links, 9 joints
Joints:
- joint button_2_0_joint: origin xyz=0 0.24119 1.269 rpy=0 0 0 -> xyz=-1.75 0.24119 1.269 rpy=0 0 0
