Commit message: Buttons URDF

File: assets/elevator.urdf (robot description, URDF)
Before this commit: robot elevator, 2 links, 1 joints
Links:
- added link button_0_0_link>, mass 0.1; collision box size=0.19 0.02 0.09; visual mesh filename=button_0_0.dae scale=1 1 1
- added link button_0_1_link>, mass 0.1; collision box size=0.19 0.02 0.09; visual mesh filename=button_0_1.dae scale=1 1 1
- added link button_1_0_link>, mass 0.1; collision box size=0.19 0.02 0.09; visual mesh filename=button_1_0.dae scale=1 1 1
- added link button_1_1_link>, mass 0.1; collision box size=0.19 0.02 0.09; visual mesh filename=button_1_1.dae scale=1 1 1
- added link button_2_0_link>, mass 0.1; collision box size=0.19 0.02 0.09; visual mesh filename=button_2_0.dae scale=1 1 1
- added link button_2_1_link>, mass 0.1; collision box size=0.19 0.02 0.09; visual mesh filename=button_2_1.dae scale=1 1 1
- added link button_3_0_link>, mass 0.1; collision box size=0.19 0.02 0.09; visual mesh filename=button_3_0.dae scale=1 1 1
- added link button_3_1_link>, mass 0.1; collision box size=0.19 0.02 0.09; visual mesh filename=button_3_1.dae scale=1 1 1
Joints:
- added joint button_0_0_joint: type prismatic, parent cabin_link, child button_0_0_link, origin xyz=X Y Z rpy=0 0 0, axis 0 -1 0, limit lower=0.0 upper=0.01 effort=20 velocity=0.2
- added joint button_0_1_joint: type prismatic, parent cabin_link, child button_0_1_link, origin xyz=X Y Z rpy=0 0 0, axis 0 -1 0, limit lower=0.0 upper=0.01 effort=20 velocity=0.2
- added joint button_1_0_joint: type prismatic, parent cabin_link, child button_1_0_link, origin xyz=X Y Z rpy=0 0 0, axis 0 -1 0, limit lower=0.0 upper=0.01 effort=20 velocity=0.2
- added joint button_1_1_joint: type prismatic, parent cabin_link, child button_1_1_link, origin xyz=X Y Z rpy=0 0 0, axis 0 -1 0, limit lower=0.0 upper=0.01 effort=20 velocity=0.2
- added joint button_2_0_joint: type prismatic, parent cabin_link, child button_2_0_link, origin xyz=X Y Z rpy=0 0 0, axis 0 -1 0, limit lower=0.0 upper=0.01 effort=20 velocity=0.2
- added joint button_2_1_joint: type prismatic, parent cabin_link, child button_2_1_link, origin xyz=X Y Z rpy=0 0 0, axis 0 -1 0, limit lower=0.0 upper=0.01 effort=20 velocity=0.2
- added joint button_3_0_joint: type prismatic, parent cabin_link, child button_3_0_link, origin xyz=X Y Z rpy=0 0 0, axis 0 -1 0, limit lower=0.0 upper=0.01 effort=20 velocity=0.2
- added joint button_3_1_joint: type prismatic, parent cabin_link, child button_3_1_link, origin xyz=X Y Z rpy=0 0 0, axis 0 -1 0, limit lower=0.0 upper=0.01 effort=20 velocity=0.2

Commit message: Fix joint

File: assets/elevator.urdf (robot description, URDF)
Before this commit: robot elevator, 10 links, 9 joints
Joints:
- joint button_0_0_joint: origin xyz=X Y Z rpy=0 0 0 -> xyz=0 0 0 rpy=0 0 0
- joint button_0_1_joint: origin xyz=X Y Z rpy=0 0 0 -> xyz=0 0 0 rpy=0 0 0
- joint button_1_0_joint: origin xyz=X Y Z rpy=0 0 0 -> xyz=0 0 0 rpy=0 0 0
- joint button_1_1_joint: origin xyz=X Y Z rpy=0 0 0 -> xyz=0 0 0 rpy=0 0 0
- joint button_2_0_joint: origin xyz=X Y Z rpy=0 0 0 -> xyz=0 0 0 rpy=0 0 0
- joint button_2_1_joint: origin xyz=X Y Z rpy=0 0 0 -> xyz=0 0 0 rpy=0 0 0
- joint button_3_0_joint: origin xyz=X Y Z rpy=0 0 0 -> xyz=0 0 0 rpy=0 0 0
- joint button_3_1_joint: origin xyz=X Y Z rpy=0 0 0 -> xyz=0 0 0 rpy=0 0 0

Commit message: Fix naming

File: assets/elevator.urdf (robot description, URDF)
Before this commit: robot elevator, 10 links, 9 joints
Links:
- removed link button_0_0_link>
- removed link button_0_1_link>
- removed link button_1_0_link>
- removed link button_1_1_link>
- removed link button_2_0_link>
- removed link button_2_1_link>
- removed link button_3_0_link>
- removed link button_3_1_link>
- added link button_0_0_link, mass 0.1; collision box size=0.19 0.02 0.09; visual mesh filename=button_0_0.dae scale=1 1 1
- added link button_0_1_link, mass 0.1; collision box size=0.19 0.02 0.09; visual mesh filename=button_0_1.dae scale=1 1 1
- added link button_1_0_link, mass 0.1; collision box size=0.19 0.02 0.09; visual mesh filename=button_1_0.dae scale=1 1 1
- added link button_1_1_link, mass 0.1; collision box size=0.19 0.02 0.09; visual mesh filename=button_1_1.dae scale=1 1 1
- added link button_2_0_link, mass 0.1; collision box size=0.19 0.02 0.09; visual mesh filename=button_2_0.dae scale=1 1 1
- added link button_2_1_link, mass 0.1; collision box size=0.19 0.02 0.09; visual mesh filename=button_2_1.dae scale=1 1 1
- added link button_3_0_link, mass 0.1; collision box size=0.19 0.02 0.09; visual mesh filename=button_3_0.dae scale=1 1 1
- added link button_3_1_link, mass 0.1; collision box size=0.19 0.02 0.09; visual mesh filename=button_3_1.dae scale=1 1 1

Commit message: Organize asset folder

File: assets/elevator.urdf (robot description, URDF)
Before this commit: robot elevator, 10 links, 9 joints
Links:
- link button_0_0_link: geometry collision box size=0.19 0.02 0.09; visual mesh filename=button.dae scale=1 1 1
- link button_0_1_link: geometry collision box size=0.19 0.02 0.09; visual mesh filename=button.dae scale=1 1 1
- link button_1_0_link: geometry collision box size=0.19 0.02 0.09; visual mesh filename=button.dae scale=1 1 1
- link button_1_1_link: geometry collision box size=0.19 0.02 0.09; visual mesh filename=button.dae scale=1 1 1
- link button_2_0_link: geometry collision box size=0.19 0.02 0.09; visual mesh filename=button.dae scale=1 1 1
- link button_2_1_link: geometry collision box size=0.19 0.02 0.09; visual mesh filename=button.dae scale=1 1 1
- link button_3_0_link: geometry collision box size=0.19 0.02 0.09; visual mesh filename=button.dae scale=1 1 1
- link button_3_1_link: geometry collision box size=0.19 0.02 0.09; visual mesh filename=button.dae scale=1 1 1
Joints:
- joint button_0_0_joint: origin xyz=0 0 0 rpy=0 0 0 -> xyz=-1.75 0.24119 1.625 rpy=0 0 0
- joint button_0_1_joint: origin xyz=0 0 0 rpy=0 0 0 -> xyz=-1.97 0.24119 1.625 rpy=0 0 0
- joint button_1_0_joint: origin xyz=0 0 0 rpy=0 0 0 -> xyz=-1.75 0.24119 1.447 rpy=0 0 0
- joint button_1_1_joint: origin xyz=0 0 0 rpy=0 0 0 -> xyz=-1.97 0.24119 1.447 rpy=0 0 0
- joint button_2_0_joint: axis 0 -1 0 -> -1.75 -1 0; origin xyz=0 0 0 rpy=0 0 0 -> xyz=-1.75 0.24119 1.269 rpy=0 0 0
- joint button_2_1_joint: origin xyz=0 0 0 rpy=0 0 0 -> xyz=-1.97 0.24119 1.269 rpy=0 0 0
- joint button_3_0_joint: origin xyz=0 0 0 rpy=0 0 0 -> xyz=-1.75 0.24119 1.091 rpy=0 0 0
- joint button_3_1_joint: origin xyz=0 0 0 rpy=0 0 0 -> xyz=-1.97 0.24119 1.091 rpy=0 0 0

Commit message: Buttons with image texture material

File: assets/elevator.urdf (robot description, URDF)
Before this commit: robot elevator, 10 links, 9 joints
Links:
- link button_0_0_link: geometry collision box size=0.19 0.02 0.09; visual mesh filename=ground_button.dae scale=1 1 1
- link button_0_1_link: geometry collision box size=0.19 0.02 0.09; visual mesh filename=2_button.dae scale=1 1 1
- link button_1_0_link: geometry collision box size=0.19 0.02 0.09; visual mesh filename=3_button.dae scale=1 1 1
- link button_1_1_link: geometry collision box size=0.19 0.02 0.09; visual mesh filename=4_button.dae scale=1 1 1
- link button_2_0_link: geometry collision box size=0.19 0.02 0.09; visual mesh filename=5_button.dae scale=1 1 1
- link button_2_1_link: geometry collision box size=0.19 0.02 0.09; visual mesh filename=6_button.dae scale=1 1 1
- link button_3_0_link: geometry collision box size=0.19 0.02 0.09; visual mesh filename=open_button.dae scale=1 1 1
- link button_3_1_link: geometry collision box size=0.19 0.02 0.09; visual mesh filename=close_button.dae scale=1 1 1

Commit message: Renamed buttons & fix

File: assets/elevator.urdf (robot description, URDF)
Before this commit: robot elevator, 10 links, 9 joints
Links:
- link button_0_0_link: geometry collision box size=0.19 0.02 0.09; visual mesh filename=button_ground.dae scale=1 1 1
- link button_0_1_link: geometry collision box size=0.19 0.02 0.09; visual mesh filename=button_2.dae scale=1 1 1
- link button_1_0_link: geometry collision box size=0.19 0.02 0.09; visual mesh filename=button_3.dae scale=1 1 1
- link button_1_1_link: geometry collision box size=0.19 0.02 0.09; visual mesh filename=button_4.dae scale=1 1 1
- link button_2_0_link: geometry collision box size=0.19 0.02 0.09; visual mesh filename=button_5.dae scale=1 1 1
- link button_2_1_link: geometry collision box size=0.19 0.02 0.09; visual mesh filename=button_6.dae scale=1 1 1
- link button_3_0_link: geometry collision box size=0.19 0.02 0.09; visual mesh filename=button_open.dae scale=1 1 1
- link button_3_1_link: geometry collision box size=0.19 0.02 0.09; visual mesh filename=button_close.dae scale=1 1 1
Joints:
- joint button_2_0_joint: axis -1.75 -1 0 -> 0 -1 0

Commit message: Reset button pos

File: assets/elevator.urdf (robot description, URDF)
Before this commit: robot elevator, 10 links, 9 joints
Links:
- link button_0_0_link: geometry collision box size=0.19 0.02 0.09; visual mesh filename=button_5.dae scale=1 1 1
- link button_0_1_link: geometry collision box size=0.19 0.02 0.09; visual mesh filename=button_6.dae scale=1 1 1
- link button_2_0_link: geometry collision box size=0.19 0.02 0.09; visual mesh filename=button_ground.dae scale=1 1 1
- link button_2_1_link: geometry collision box size=0.19 0.02 0.09; visual mesh filename=button_2.dae scale=1 1 1

Commit message: Modified door 2

File: assets/elevator.urdf (robot description, URDF)
Before this commit: robot elevator, 10 links, 9 joints
Joints:
- joint door2_joint: origin xyz=0 0 0 rpy=0 0 0 -> xyz=-0.22 0.09 1.37 rpy=0 0 0

Commit message: Fix door axis direction

File: assets/elevator.urdf (robot description, URDF)
Before this commit: robot elevator, 10 links, 9 joints
Joints:
- joint door2_joint: axis 1 0 0 -> -1 0 0

Commit message: Test

File: assets/elevator.urdf (robot description, URDF)
Before this commit: robot elevator, 10 links, 9 joints
Joints:
- joint door2_joint: axis -1 0 0 -> 1 0 0; limit lower=-0.5 upper=0.0 effort=200 velocity=0.5 -> lower=0.0 upper=0.5 effort=200 velocity=0.5

Commit message: Remove door 2 from URDF and set as standalone animation

File: assets/elevator.urdf (robot description, URDF)
Before this commit: robot elevator, 10 links, 9 joints
Links:
- removed link door2_link
Joints:
- removed joint door2_joint

Commit message: Modified the panel

File: assets/elevator.urdf (robot description, URDF)
Before this commit: robot elevator, 9 links, 8 joints
Links:
- added link panel_link, mass 50.0; collision box size=0.0 0.0 0.0; visual mesh filename=elevator_panel.dae scale=1 1 1

Commit message: Omit panel collision

File: assets/elevator.urdf (robot description, URDF)
Before this commit: robot elevator, 10 links, 8 joints
Links:
- link panel_link: geometry visual mesh filename=elevator_panel.dae scale=1 1 1

Commit message: Small collision instead

File: assets/elevator.urdf (robot description, URDF)
Before this commit: robot elevator, 10 links, 8 joints
Links:
- link panel_link: geometry collision box size=0.1 0.1 0.1; visual mesh filename=elevator_panel.dae scale=1 1 1

Commit message: Add link for panel

File: assets/elevator.urdf (robot description, URDF)
Before this commit: robot elevator, 10 links, 8 joints
Joints:
- added joint panel_joint: type fixed, parent cabin_link, child panel_link, origin xyz=0 0 0 rpy=0 0 0

Commit message: Add door2 as static joint

File: assets/elevator.urdf (robot description, URDF)
Before this commit: robot elevator, 10 links, 9 joints
Links:
- added link door2_link, mass 5.0; collision box size=0.1 0.1 0.1; visual mesh filename=door2.dae scale=1 1 1
Joints:
- added joint door2_joint: type prismatic, parent cabin_link, child door2_link, origin xyz=-0.22 0.09 1.37 rpy=0 0 0

Commit message: Add door1 as prismatic joint

File: assets/elevator.urdf (robot description, URDF)
Before this commit: robot elevator, 11 links, 10 joints
Links:
- added link door1_link, mass 5.0; collision box size=0.1 0.1 0.1; visual mesh filename=door1.dae scale=1 1 1
Joints:
- added joint door1_joint: type prismatic, parent cabin_link, child door1_link, origin xyz=0.74 0.11 1.37 rpy=0 0 0, axis -1 0 0, limit lower=0.0 upper=0.8 effort=20 velocity=0.2

Commit message: elevator wall

File: assets/elevator.urdf (robot description, URDF)
Before this commit: robot elevator, 12 links, 11 joints
Links:
- link cabin_link: geometry collision box size=4.2356 0.2952 3.2904; visual mesh filename=elevator_wall.dae scale=1 1 1

Commit message: New button positions & panel

File: assets/elevator.urdf (robot description, URDF)
Before this commit: robot elevator, 12 links, 11 joints
Joints:
- joint button_0_0_joint: origin xyz=-1.75 0.24119 1.625 rpy=0 0 0 -> xyz=-1.75 0.34158 1.625 rpy=0 0 0
- joint button_0_1_joint: origin xyz=-1.97 0.24119 1.625 rpy=0 0 0 -> xyz=-1.97 0.34158 1.625 rpy=0 0 0
- joint button_1_0_joint: origin xyz=-1.75 0.24119 1.447 rpy=0 0 0 -> xyz=-1.75 0.34158 1.447 rpy=0 0 0
- joint button_1_1_joint: origin xyz=-1.97 0.24119 1.447 rpy=0 0 0 -> xyz=-1.97 0.34158 1.447 rpy=0 0 0
- joint button_2_0_joint: origin xyz=-1.75 0.24119 1.269 rpy=0 0 0 -> xyz=-1.75 0.34158 1.269 rpy=0 0 0
- joint button_2_1_joint: origin xyz=-1.97 0.24119 1.269 rpy=0 0 0 -> xyz=-1.97 0.34158 1.269 rpy=0 0 0
- joint button_3_0_joint: origin xyz=-1.75 0.24119 1.091 rpy=0 0 0 -> xyz=-1.75 0.34158 1.091 rpy=0 0 0
- joint button_3_1_joint: origin xyz=-1.97 0.24119 1.091 rpy=0 0 0 -> xyz=-1.97 0.34158 1.091 rpy=0 0 0
